File: scheamt.kicad_sch (KiCad schematic)
At the start: 6 parts, among them J1 Raspberry_Pi_2_3, M1 Motor_Servo, M2 Motor_Servo, M3 Motor_Servo

Commit message: Dodanie, Line i Neutral
Parts:
- M1, M2, M3: value Motor_Servo -> SG 90
Connections:
- net LINE: now reaches PS1.1 (AC/L)
- net NEUT: now reaches PS1.2 (AC/N)

Commit message: Add files via upload
Parts:
- added U1: Flir_LEPTON, symbol Sensor_Optical:Flir_LEPTON
- .: renamed from PS1; value IRM-20-5 -> RS-25-5; footprint Converter_ACDC:Converter_ACDC_MeanWell_IRM-20-xx_THT -> Converter_ACDC_MeanWell_RS-25-5
- J1: value Raspberry_Pi_2_3 -> Raspberry Pi 4 model B
- M1, M2, M3: value SG 90 -> Microservo SG90
Connections:
- net at J1.6 (GND), M1.3 (-), M2.3 (-)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: now also ..5 (-Vo); no longer ..3 (-Vo)
- net LINE: no longer names the net of ..1 (AC/L)
- net NEUT: no longer names the net of ..2 (AC/N)
- new net: J1. (SDA), U1. (SDA) (x10)
Other:
- note added: "Kamera HD B OV5647 5Mpx - z regulacją ostrości dla Raspberry Pi - Waveshare 8193"
- moved on the sheet: ., F1, M1, M2, M3
